File: rudolph_led_driver.kicad_sch (KiCad schematic)
At the start: 33 parts, among them J1 Conn_01x02_Female, J2 USB_B_Micro, J3 Conn_01x02_Male, Q1 S8050, Q2 2SC1815, Q3 2SC1815, Q4 S8050, Q5 S8050, Q6 2SC1815, SW1 ON/OFF, U1 LM809, U2 LP2980-ADJ, U3 MCP73831-2-OT

Commit message: Minor tweaks to the voltage reference generator
Parts:
- added C1: 4.7uF, Capacitor_SMD:C_0805_2012Metric_Pad1.18x1.45mm_HandSolder, symbol Device:C
- C3: renamed from C1; value 2.2uF -> 4.7uF
- U1: value LM809 -> BD49K33G; Manufacturer (none) -> Rohm
- renumbered C3 to C4, DL2 to DL1, DL1 to DL2, J2 to J1, J1 to J2, Q3 to Q1, Q4 to Q2, Q1 to Q3, Q2 to Q4, R7 to R1, R11 to R10, R5 to R11, R1 to R2, R4 to R3, R3 to R4, R6 to R5, R8 to R6, R10 to R7, R9 to R8, R2 to R9
Connections:
- net +BATT: now also SW1.1 (A); no longer R2.1, U1.3 (VCC), U2.1 (VIN)
- net GND: now also C1.2
- net at SW1.2 (B): now also R2.1, U1.3 (VCC), U2.1 (VIN), C1.1; no longer U2.3 (ON/~{OFF})
- net at R2.2, U1.2 (~{RESET}): now also U2.3 (ON/~{OFF}); no longer SW1.1 (A)
Other:
- note added: "Minimum battery voltage: 3.3V Populate R1 if using an open-drain voltage supervisor"
- moved on the sheet: R2, R3, R4, SW1, U1, U2
